File: eda/ATX2PCjr/ATX2PCjr.sch (KiCad schematic (older format))
At the start: 4 parts, among them J1 ATX Connector, J2 PCjr Card Edge, J3 Power Switch Header, J4 Fan Header

Commit message: Board version 1.1
Parts:
- added J5: Floppy Power, ATX2PCjr:Mate-N-Lok Vertical, symbol Connector_Generic:Conn_01x04
Connections:
- wire segments 35 -> 41
Changed lines of the file:
@@
 Text Label 5250 4200 0    50   ~ 0
 PS-ON
+$Comp
+L Connector_Generic:Conn_01x04 J5
+U 1 1 5B6FB298
+P 5650 1550
+F 0 "J5" H 5729 1542 50  0000 L CNN
+F 1 "Floppy Power" H 5729 1451 50  0000 L CNN
+F 2 "ATX2PCjr:Mate-N-Lok Vertical" H 5650 1550 50  0001 C CNN
+F 3 "~" H 5650 1550 50  0001 C CNN
+	1    5650 1550
+	1    0    0    -1
+$EndComp
+Wire Wire Line
+	5250 1550 5250 1650
+Wire Wire Line
+	5250 1650 5450 1650
+Wire Wire Line
+	5250 1550 5450 1550
+Wire Wire Line
+	5450 1550 5500 1550
+Text Label 5250 1550 0    50   ~ 0
+GND
+Wire Wire Line
+	5150 1750 5450 1750
+Wire Wire Line
+	5150 1450 5450 1450
+Text Label 5150 1750 0    50   ~ 0
++12V
+Text Label 5150 1450 0    50   ~ 0
++5V
+Connection ~ 5450 1550
 $EndSCHEMATC

Commit message: Updated to v1.11 to fix minor issues
Parts:
- added J6: Fan Header, Connector_PinHeader_2.54mm:PinHeader_1x03_P2.54mm_Vertical, symbol Connector_Generic_MountingPin:Conn_01x03_MountingPin
Connections:
- wire segments 41 -> 45
Changed lines of the file:
@@
 +5V
 Connection ~ 5450 1550
+$Comp
+L Connector_Generic_MountingPin:Conn_01x03_MountingPin J6
+U 1 1 5B909F5C
+P 6950 2200
+F 0 "J6" H 7038 2166 50  0000 L CNN
+F 1 "Fan Header" H 7038 2075 50  0000 L CNN
+F 2 "Connector_PinHeader_2.54mm:PinHeader_1x03_P2.54mm_Vertical" H 6950 2200 50  0001 C CNN
+F 3 "~" H 6950 2200 50  0001 C CNN
+	1    6950 2200
+	1    0    0    -1
+$EndComp
+Wire Wire Line
+	6750 2300 6350 2300
+Wire Wire Line
+	6350 2300 6350 2100
+Wire Wire Line
+	6350 2100 6750 2100
+Wire Wire Line
+	6750 2200 6550 2200
+Text Label 6550 2100 0    50   ~ 0
+GND
+Text Label 6550 2200 0    50   ~ 0
++12V
 $EndSCHEMATC

Commit message: MiniFit Jr Vias and Panel Holes
Parts:
- J1: footprint Connector_Molex:Molex_Mini-Fit_Jr_5566-20A2_2x10_P4.20mm_Vertical -> ATX2PCjr:Molex_Mini-Fit_Jr_5566-20A2_2x10_P4.20mm_Vertical-LARGE
Changed lines of the file:
@@
 F 0 "J1" H 3188 3273 50  0000 L CNN
 F 1 "ATX Connector" H 3188 3364 50  0000 L CNN
-F 2 "Connector_Molex:Molex_Mini-Fit_Jr_5566-20A2_2x10_P4.20mm_Vertical" H 3100 3450 50  0001 C CNN
+F 2 "ATX2PCjr:Molex_Mini-Fit_Jr_5566-20A2_2x10_P4.20mm_Vertical-LARGE" H 3100 3450 50  0001 C CNN
 F 3 "~" H 3100 3450 50  0001 C CNN
 	1    3100 3450
